File: kicad/k1-aioc/k1-aioc.kicad_pcb (KiCad board)
At the start: 2 copper layers, 21 x 31.5 mm, 47 parts, among them J1 12401832E402A, J2 Conn_01x07_Male, Q1 BC847BS, U1 MIC5330-SSYML, U2 STM32F373CBTx, Y1 8MHz/20pF

Commit message: convert TRS plugs to 2.54mm pitch screw terminals
Parts:
- added J3: Conn_01x03, TerminalBlock:TerminalBlock_Xinya_XY308-2.54-3P_1x03_P2.54mm_Horizontal, F.Cu at (128.5, 108.5)
- added J4: Conn_01x03, TerminalBlock:TerminalBlock_Xinya_XY308-2.54-3P_1x03_P2.54mm_Horizontal, F.Cu at (128.5, 98.6)
Routing:
- net /RADIO-RX-PTT1: track 30.0 -> 43.3 mm
- net /RADIO-VP-PTT2: track 4.77 -> 12.4 mm
- net /RADIO-MIC: track 2.93 -> 9.61 mm
- net /RADIO-SPK: track 2.01 -> 6.60 mm
- net /RADIO-TX: track 24.2 -> 22.3 mm, vias 2 -> 1
- removed copper zone on F.Cu, net /RADIO-MIC
- removed copper zone on B.Cu, net /RADIO-RX-PTT1
- removed copper zone on F.Cu, net /RADIO-SPK
- removed copper zone on F.Cu, net /RADIO-TX
- removed copper zone on F.Cu, net /RADIO-VP-PTT2
Other:
- board size 21 x 31.5 mm -> 30 x 31.5 mm
