File: kicad/k1-aioc/k1-aioc.kicad_sch (KiCad schematic)
At the start: 46 parts, among them J1 12401832E402A, J2 Conn_01x07_Male, Q1 BC847BS, U1 MIC5330-SSYML, U2 STM32F373CBTx, Y1 8MHz/20pF

Commit message: convert TRS plugs to 2.54mm pitch screw terminals
Parts:
- added J3, J4: Conn_01x03, TerminalBlock:TerminalBlock_Xinya_XY308-2.54-3P_1x03_P2.54mm_Horizontal, symbol Connector_Generic:Conn_01x03
Connections:
- net GND: now also J4.2 (Pin_2)
- net RADIO-MIC: now also J3.1 (Pin_1)
- net RADIO-RX-PTT1: now also J3.2 (Pin_2)
- net RADIO-SPK: now also J4.3 (Pin_3)
- net RADIO-TX: now also J4.1 (Pin_1)
- net RADIO-VP-PTT2: now also J3.3 (Pin_3)
